File: Energieplatine/Energieplatine.kicad_pcb (KiCad board)
At the start: 2 copper layers, 90.2 x 44.4 mm, 40 parts, among them J2 Conn_01x02_Pin, J3 Conn_01x02_Pin, J4 Conn_02x07_Odd_Even, J5 Conn_01x02_Pin, J6 Conn_01x02_Pin, J7 USB3_A, Q1 IRF9540N, Q2 IRF9540N, Q3 IRF540N, U1 4027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

Commit message: Added Logo on Silkscreen
Logo und Platinenbeschriftung hinzugefügt
Parts:
- added G***: LOGO, LOGO, F.Cu at (140.7, 114.4)
Other:
- board text added: "Tutorenprojekt 2024 Energieplatine"
